Commit message: fix minor bugs

File: urdf/kwr75.ros2_control.xacro (robot description, xacro)
@@ -2,33 +2,33 @@
 <robot xmlns:xacro="http://www.ros.org/wiki/xacro">
   <xacro:macro name="kwr75_force_sensor_ros2_control" params="name prefix com_port:=/dev/ttyUSB0 use_mock_hardware:=false mock_sensor_commands:=false">
-    <ros2_control name="${name}" type="sensor">
-      <hardware>
-        <xacro:if value="${use_mock_hardware}">
-          <plugin>mock_components/GenericSystem</plugin>
-          <param name="mock_sensor_commands">${mock_sensor_commands}</param>
-          <param name="position_state_following_offset">0.0</param>
-        </xacro:if>
-        <xacro:unless value="${use_mock_hardware}">
+    <xacro:unless value="${use_mock_hardware}">
+      <ros2_control name="${name}" type="sensor">
+        <hardware>
+          <!-- <xacro:if value="${use_mock_hardware}">
+            <plugin>mock_components/GenericSystem</plugin>
+            <param name="mock_sensor_commands">${mock_sensor_commands}</param>
+            <param name="position_state_following_offset">0.0</param>
+          </xacro:if> -->
           <plugin>kwr75_force_sensor/KWR75ForceSensorHardwareInterface</plugin>
           <param name="com_port">${com_port}</param>
           <param name="baud_rate">460800</param>
-        </xacro:unless>
-      </hardware>
-      <sensor name="${prefix}kwr75_force_sensor">
-        <state_interface name="force.x"/>
-        <state_interface name="force.y"/>
-        <state_interface name="force.z"/>
-        <state_interface name="torque.x"/>
-        <state_interface name="torque.y"/>
-        <state_interface name="torque.z"/>
-        <param name="frame_id">${prefix}fts_link</param>
-        <param name="fx_range">100</param>
-        <param name="fy_range">100</param>
-        <param name="fz_range">100</param>
-        <param name="tx_range">15</param>
-        <param name="ty_range">15</param>
-        <param name="tz_range">15</param>
-      </sensor>
-    </ros2_control>
+        </hardware>
+        <sensor name="${prefix}kwr75_force_sensor">
+          <state_interface name="force.x"/>
+          <state_interface name="force.y"/>
+          <state_interface name="force.z"/>
+          <state_interface name="torque.x"/>
+          <state_interface name="torque.y"/>
+          <state_interface name="torque.z"/>
+          <param name="frame_id">${prefix}fts_link</param>
+          <param name="fx_range">100</param>
+          <param name="fy_range">100</param>
+          <param name="fz_range">100</param>
+          <param name="tx_range">15</param>
+          <param name="ty_range">15</param>
+          <param name="tz_range">15</param>
+        </sensor>
+      </ros2_control>
+    </xacro:unless>
   </xacro:macro>
 </robot>

File: urdf/kwr75_macro.xacro (robot description, xacro)
@@ -14,5 +14,5 @@
       </inertial>
       <visual>
-        <origin xyz="0 0 0" rpy="${-pi/2} 0 0"/>
+        <origin xyz="0 0 0.013" rpy="${-pi/2} 0 0"/>
         <geometry>
           <mesh filename="package://kwr75_force_sensor_ros2/meshes/kwr75.dae" scale="0.001 0.001 0.001"/>
